Commit message: cart finished

File: src/my_robot/urdf/my_robot.xacro (robot description, xacro)
@@ -8,4 +8,70 @@
     <child link="chassis" />
   </joint>
+  <joint name="robot_footprint_joint2" type="fixed">
+    <origin xyz="0 0 0" rpy="0 0 0" />
+    <parent link="robot_footprint"/>
+    <child link="cart_body" />
+  </joint>
+  <link name="cart_body">
+    <pose> 0 0 0.3 0 0 0 </pose>
+    <inertial>
+      <mass value="15.0"/>
+      <origin xyz="0.0 0 0" rpy=" 0 0 0"/>
+      <inertia
+          ixx="0.166667" ixy="0" ixz="0"
+          iyy="0.166667" iyz="0"
+          izz="0.166667"
+      />
+    </inertial>
+    <collision name='cart_collision'>
+      <origin xyz="0 0 0.4" rpy=" 0 0 0"/>
+      <geometry>
+        <box size="1 0.6 0.8"/>
+      </geometry>
+    </collision>
+    <visual name='cart_visual_button'>
+      <origin xyz="0 0 0.3" rpy=" 0 0 0"/>
+      <geometry>
+        <box size="1 0.6 0.05"/>
+      </geometry>
+      <origin xyz="-0.5 -0.25 0" rpy=" 0 0 0"/>
+    </visual>
+    <visual name='cart_visual_middle'>
+      <origin xyz="0 0 0.5" rpy=" 0 0 0"/>
+      <geometry>
+        <box size="1 0.6 0.05"/>
+      </geometry>
+    </visual>
+    <visual name='cart_visual_top'>
+      <origin xyz="0 0 0.7" rpy=" 0 0 0"/>
+      <geometry>
+        <box size="1 0.6 0.05"/>
+      </geometry>
+    </visual>
+    <visual name='cart_visual_fl'>
+      <origin xyz="0.5 0.25 0.4" rpy=" 0 0 0"/>
+      <geometry>
+        <box size="0.1 0.1 0.8"/>
+      </geometry>
+    </visual>
+    <visual name='cart_visual_bl'>
+      <origin xyz="-0.5 0.25 0.4" rpy=" 0 0 0"/>
+      <geometry>
+        <box size="0.1 0.1 0.8"/>
+      </geometry>
+    </visual>
+    <visual name='cart_visual_fr'>
+      <origin xyz="0.5 -0.25 0.4" rpy=" 0 0 0"/>
+      <geometry>
+        <box size="0.1 0.1 0.8"/>
+      </geometry>
+    </visual>
+    <visual name='cart_visual_br'>
+      <origin xyz="-0.5 -0.25 0.4" rpy=" 0 0 0"/>
+      <geometry>
+        <box size="0.1 0.1 0.8"/>
+      </geometry>
+    </visual>
+  </link>
   <link name='chassis'>
     <pose>0 0 0.1 0 0 0</pose>
@@ -22,5 +88,5 @@
       <origin xyz="0 0 0" rpy=" 0 0 0"/>
       <geometry>
-        <box size=".4 .2 .1"/>
+        <box size="1.2 0.8 0.05"/>
       </geometry>
     </collision>
@@ -28,29 +94,5 @@
       <origin xyz="0 0 0" rpy=" 0 0 0"/>
       <geometry>
-        <box size=".4 .2 .1"/>
-      </geometry>
-    </visual>
-    <collision name='back_caster_collision'>
-      <origin xyz="-0.15 0 -0.05" rpy=" 0 0 0"/>
-      <geometry>
-        <sphere radius="0.0499"/>
-      </geometry>
-    </collision>
-    <visual name='back_caster_visual'>
-      <origin xyz="-0.15 0 -0.05" rpy=" 0 0 0"/>
-      <geometry>
-        <sphere radius="0.05"/>
-      </geometry>
-    </visual>
-    <collision name='front_caster_collision'>
-      <origin xyz="0.15 0 -0.05" rpy=" 0 0 0"/>
-      <geometry>
-        <sphere radius="0.0499"/>
-      </geometry>
-    </collision>
-    <visual name='front_caster_visual'>
-      <origin xyz="0.15 0 -0.05" rpy=" 0 0 0"/>
-      <geometry>
-        <sphere radius="0.05"/>
+        <box size="1.2 0.8 0.05"/>
       </geometry>
     </visual>
@@ -102,6 +144,52 @@
     </visual>
   </link>
+<link name='back_left_wheel'>
+    <inertial>
+      <mass value="5.0"/>
+      <origin xyz="0.0 0 0" rpy=" 0 1.5707 1.5707"/>
+      <inertia
+          ixx="0.1" ixy="0" ixz="0"
+          iyy="0.1" iyz="0"
+          izz="0.1"
+      />
+    </inertial>
+    <collision name='back_left_whee_collision'>
+      <origin xyz="0 0 0" rpy="0 1.5707 1.5707"/>
+      <geometry>
+        <cylinder  radius="0.1" length="0.05"/>
+      </geometry>
+    </collision>
+    <visual name='back_left_wheel_visual'>
+      <origin xyz="0 0 0" rpy=" 0 1.5707 1.5707"/>
+      <geometry>
+        <cylinder  radius="0.1" length="0.05"/>
+      </geometry>
+    </visual>
+  </link>
+<link name='back_right_wheel'>
+    <inertial>
+      <mass value="5.0"/>
+      <origin xyz="0.0 0 0" rpy=" 0 1.5707 1.5707"/>
+      <inertia
+          ixx="0.1" ixy="0" ixz="0"
+          iyy="0.1" iyz="0"
+          izz="0.1"
+      />
+    </inertial>
+    <collision name='back_right_wheel_collision'>
+      <origin xyz="0 0 0" rpy="0 1.5707 1.5707"/>
+      <geometry>
+        <cylinder  radius="0.1" length="0.05"/>
+      </geometry>
+    </collision>
+    <visual name='back_right_wheel_visual'>
+      <origin xyz="0 0 0" rpy=" 0 1.5707 1.5707"/>
+      <geometry>
+        <cylinder  radius="0.1" length="0.05"/>
+      </geometry>
+    </visual>
+  </link>
   <joint type="continuous" name="left_wheel_hinge">
-    <origin xyz="0 0.15 0" rpy="0 0 0"/>
+    <origin xyz="0.6 0.5 0" rpy="0 0 0"/>
     <child link="left_wheel"/>
     <parent link="chassis"/>
@@ -111,5 +199,5 @@
   </joint>
   <joint type="continuous" name="right_wheel_hinge">
-    <origin xyz="0 -0.15 0" rpy="0 0 0"/>
+    <origin xyz="0.6 -0.5 0" rpy="0 0 0"/>
     <child link="right_wheel"/>
     <parent link="chassis"/>
@@ -117,4 +205,20 @@
     <limit effort="10000" velocity="1000"/>
     <dynamics damping="1.0" friction="1.0"/>
+  </joint>
+  <joint type="continuous" name="back_left_wheel_hinge">
+    <origin xyz="-0.6 0.5 0" rpy="0 0 0"/>
+    <child link="back_left_wheel"/>
+    <parent link="chassis"/>
+    <axis xyz="0 1 0" rpy="0 0 0"/>
+    <limit effort="10000" velocity="1000"/>
+    <dynamics damping="1.0" friction="0.1"/>
+  </joint>
+  <joint type="continuous" name="back_right_wheel_hinge">
+    <origin xyz="-0.6 -0.5 0" rpy="0 0 0"/>
+    <child link="back_right_wheel"/>
+    <parent link="chassis"/>
+    <axis xyz="0 1 0" rpy="0 0 0"/>
+    <limit effort="10000" velocity="1000"/>
+    <dynamics damping="1.0" friction="0.1"/>
   </joint>
   <link name='camera'>
@@ -145,5 +249,5 @@
   </link>
   <joint type="fixed" name="camera_joint">
-    <origin xyz="0.2 0 0" rpy="0 0 0"/>
+    <origin xyz="0.60 0 0" rpy="0 0 0"/>
     <child link="camera"/>
     <parent link="chassis"/>
@@ -177,5 +281,5 @@
   </link>
   <joint type="fixed" name="hokuyo_joint">
-    <origin xyz="0.15 0 .1" rpy="0 0 0"/>
+    <origin xyz="0.6 0 .06" rpy="0 0 0"/>
     <child link="hokuyo"/>
     <parent link="chassis"/>

Commit message: finished chase it

File: src/my_robot/urdf/my_robot.xacro (robot description, xacro)
@@ -88,5 +88,5 @@
       <origin xyz="0 0 0" rpy=" 0 0 0"/>
       <geometry>
-        <box size="1.2 0.8 0.05"/>
+        <box size="1.1 0.6 0.05"/>
       </geometry>
     </collision>
@@ -94,5 +94,5 @@
       <origin xyz="0 0 0" rpy=" 0 0 0"/>
       <geometry>
-        <box size="1.2 0.8 0.05"/>
+        <box size="1.1 0.6 0.05"/>
       </geometry>
     </visual>
@@ -191,5 +191,5 @@
   </link>
   <joint type="continuous" name="left_wheel_hinge">
-    <origin xyz="0.6 0.5 0" rpy="0 0 0"/>
+    <origin xyz="0.5 0.4 0" rpy="0 0 0"/>
     <child link="left_wheel"/>
     <parent link="chassis"/>
@@ -199,5 +199,5 @@
   </joint>
   <joint type="continuous" name="right_wheel_hinge">
-    <origin xyz="0.6 -0.5 0" rpy="0 0 0"/>
+    <origin xyz="0.5 -0.4 0" rpy="0 0 0"/>
     <child link="right_wheel"/>
     <parent link="chassis"/>
@@ -207,18 +207,18 @@
   </joint>
   <joint type="continuous" name="back_left_wheel_hinge">
-    <origin xyz="-0.6 0.5 0" rpy="0 0 0"/>
+    <origin xyz="-0.5 0.4 0" rpy="0 0 0"/>
     <child link="back_left_wheel"/>
     <parent link="chassis"/>
     <axis xyz="0 1 0" rpy="0 0 0"/>
     <limit effort="10000" velocity="1000"/>
-    <dynamics damping="1.0" friction="0.1"/>
+    <dynamics damping="1.0" friction="1.0"/>
   </joint>
   <joint type="continuous" name="back_right_wheel_hinge">
-    <origin xyz="-0.6 -0.5 0" rpy="0 0 0"/>
+    <origin xyz="-0.5 -0.4 0" rpy="0 0 0"/>
     <child link="back_right_wheel"/>
     <parent link="chassis"/>
     <axis xyz="0 1 0" rpy="0 0 0"/>
     <limit effort="10000" velocity="1000"/>
-    <dynamics damping="1.0" friction="0.1"/>
+    <dynamics damping="1.0" friction="1.0"/>
   </joint>
   <link name='camera'>
@@ -249,5 +249,5 @@
   </link>
   <joint type="fixed" name="camera_joint">
-    <origin xyz="0.60 0 0" rpy="0 0 0"/>
+    <origin xyz="0.55 0 0" rpy="0 0 0"/>
     <child link="camera"/>
     <parent link="chassis"/>
@@ -281,5 +281,5 @@
   </link>
   <joint type="fixed" name="hokuyo_joint">
-    <origin xyz="0.6 0 .06" rpy="0 0 0"/>
+    <origin xyz="0.5 0 .06" rpy="0 0 0"/>
     <child link="hokuyo"/>
     <parent link="chassis"/>

Commit message: final chaseit2

File: src/my_robot/urdf/my_robot.xacro (robot description, xacro)
@@ -14,12 +14,12 @@
   </joint>
   <link name="cart_body">
-    <pose> 0 0 0.3 0 0 0 </pose>
-    <inertial>
-      <mass value="15.0"/>
-      <origin xyz="0.0 0 0" rpy=" 0 0 0"/>
-      <inertia
-          ixx="0.166667" ixy="0" ixz="0"
-          iyy="0.166667" iyz="0"
-          izz="0.166667"
+    <pose> 0 0 0 0 0 0 </pose>
+    <inertial>
+      <mass value="5.0"/>
+      <origin xyz="0 0 0" rpy=" 0 0 0"/>
+      <inertia
+          ixx="0.5" ixy="0" ixz="0"
+          iyy="0.3" iyz="0"
+          izz="0.4"
       />
     </inertial>
@@ -77,10 +77,10 @@
     <pose>0 0 0.1 0 0 0</pose>
     <inertial>
-      <mass value="15.0"/>
-      <origin xyz="0.0 0 0" rpy=" 0 0 0"/>
-      <inertia
-          ixx="0.1" ixy="0" ixz="0"
-          iyy="0.1" iyz="0"
-          izz="0.1"
+      <mass value="5.0"/>
+      <origin xyz="0.0 0 0" rpy=" 0 0 0"/>
+      <inertia
+          ixx="0.55" ixy="0" ixz="0"
+          iyy="0.3" iyz="0"
+          izz="0.025"
       />
     </inertial>
@@ -100,10 +100,10 @@
   <link name='left_wheel'>
     <inertial>
-      <mass value="5.0"/>
+      <mass value="0.2"/>
       <origin xyz="0.0 0 0" rpy=" 0 1.5707 1.5707"/>
       <inertia
-          ixx="0.1" ixy="0" ixz="0"
-          iyy="0.1" iyz="0"
-          izz="0.1"
+          ixx="0.05" ixy="0" ixz="0"
+          iyy="0.025" iyz="0"
+          izz="0.05"
       />
     </inertial>
@@ -113,4 +113,14 @@
         <cylinder  radius="0.1" length="0.05"/>
       </geometry>
+      <surface>
+          <friction>
+            <ode>
+              <mu>1</mu>
+              <mu2>1</mu2>
+              <slip1>0.5</slip1>
+              <slip2>0</slip2>
+            </ode>
+          </friction>
+        </surface>
     </collision>
     <visual name='left_wheel_visual'>
@@ -123,10 +133,10 @@
 <link name='right_wheel'>
     <inertial>
-      <mass value="5.0"/>
+      <mass value="0.2"/>
       <origin xyz="0.0 0 0" rpy=" 0 1.5707 1.5707"/>
       <inertia
-          ixx="0.1" ixy="0" ixz="0"
-          iyy="0.1" iyz="0"
-          izz="0.1"
+          ixx="0.05" ixy="0" ixz="0"
+          iyy="0.025" iyz="0"
+          izz="0.05"
       />
     </inertial>
@@ -136,4 +146,14 @@
         <cylinder  radius="0.1" length="0.05"/>
       </geometry>
+      <surface>
+          <friction>
+            <ode>
+              <mu>1</mu>
+              <mu2>1</mu2>
+              <slip1>0.5</slip1>
+              <slip2>0</slip2>
+            </ode>
+          </friction>
+        </surface>
     </collision>
     <visual name='right_wheel_visual'>
@@ -146,10 +166,10 @@
 <link name='back_left_wheel'>
     <inertial>
-      <mass value="5.0"/>
+      <mass value="0.2"/>
       <origin xyz="0.0 0 0" rpy=" 0 1.5707 1.5707"/>
       <inertia
-          ixx="0.1" ixy="0" ixz="0"
-          iyy="0.1" iyz="0"
-          izz="0.1"
+          ixx="0.05" ixy="0" ixz="0"
+          iyy="0.025" iyz="0"
+          izz="0.05"
       />
     </inertial>
@@ -159,4 +179,14 @@
         <cylinder  radius="0.1" length="0.05"/>
       </geometry>
+      <surface>
+          <friction>
+            <ode>
+              <mu>1</mu>
+              <mu2>1</mu2>
+              <slip1>0.5</slip1>
+              <slip2>0</slip2>
+            </ode>
+          </friction>
+        </surface>
     </collision>
     <visual name='back_left_wheel_visual'>
@@ -169,10 +199,10 @@
 <link name='back_right_wheel'>
     <inertial>
-      <mass value="5.0"/>
+      <mass value="0.2"/>
       <origin xyz="0.0 0 0" rpy=" 0 1.5707 1.5707"/>
       <inertia
-          ixx="0.1" ixy="0" ixz="0"
-          iyy="0.1" iyz="0"
-          izz="0.1"
+          ixx="0.05" ixy="0" ixz="0"
+          iyy="0.025" iyz="0"
+          izz="0.05"
       />
     </inertial>
@@ -182,4 +212,14 @@
         <cylinder  radius="0.1" length="0.05"/>
       </geometry>
+      <surface>
+          <friction>
+            <ode>
+              <mu>1</mu>
+              <mu2>1</mu2>
+              <slip1>0.5</slip1>
+              <slip2>0</slip2>
+            </ode>
+          </friction>
+        </surface>
     </collision>
     <visual name='back_right_wheel_visual'>
@@ -191,5 +231,5 @@
   </link>
   <joint type="continuous" name="left_wheel_hinge">
-    <origin xyz="0.5 0.4 0" rpy="0 0 0"/>
+    <origin xyz="0.45 0.35 0" rpy="0 0 0"/>
     <child link="left_wheel"/>
     <parent link="chassis"/>
@@ -199,5 +239,5 @@
   </joint>
   <joint type="continuous" name="right_wheel_hinge">
-    <origin xyz="0.5 -0.4 0" rpy="0 0 0"/>
+    <origin xyz="0.45 -0.35 0" rpy="0 0 0"/>
     <child link="right_wheel"/>
     <parent link="chassis"/>
@@ -207,5 +247,5 @@
   </joint>
   <joint type="continuous" name="back_left_wheel_hinge">
-    <origin xyz="-0.5 0.4 0" rpy="0 0 0"/>
+    <origin xyz="-0.45 0.35 0" rpy="0 0 0"/>
     <child link="back_left_wheel"/>
     <parent link="chassis"/>
@@ -215,5 +255,5 @@
   </joint>
   <joint type="continuous" name="back_right_wheel_hinge">
-    <origin xyz="-0.5 -0.4 0" rpy="0 0 0"/>
+    <origin xyz="-0.45 -0.35 0" rpy="0 0 0"/>
     <child link="back_right_wheel"/>
     <parent link="chassis"/>

Commit message: amcl finish

File: src/my_robot/urdf/my_robot.xacro (robot description, xacro)
@@ -197,37 +197,4 @@
     </visual>
   </link>
-<link name='back_right_wheel'>
-    <inertial>
-      <mass value="0.2"/>
-      <origin xyz="0.0 0 0" rpy=" 0 1.5707 1.5707"/>
-      <inertia
-          ixx="0.05" ixy="0" ixz="0"
-          iyy="0.025" iyz="0"
-          izz="0.05"
-      />
-    </inertial>
-    <collision name='back_right_wheel_collision'>
-      <origin xyz="0 0 0" rpy="0 1.5707 1.5707"/>
-      <geometry>
-        <cylinder  radius="0.1" length="0.05"/>
-      </geometry>
-      <surface>
-          <friction>
-            <ode>
-              <mu>1</mu>
-              <mu2>1</mu2>
-              <slip1>0.5</slip1>
-              <slip2>0</slip2>
-            </ode>
-          </friction>
-        </surface>
-    </collision>
-    <visual name='back_right_wheel_visual'>
-      <origin xyz="0 0 0" rpy=" 0 1.5707 1.5707"/>
-      <geometry>
-        <cylinder  radius="0.1" length="0.05"/>
-      </geometry>
-    </visual>
-  </link>
   <joint type="continuous" name="left_wheel_hinge">
     <origin xyz="0.45 0.35 0" rpy="0 0 0"/>
@@ -247,14 +214,6 @@
   </joint>
   <joint type="continuous" name="back_left_wheel_hinge">
-    <origin xyz="-0.45 0.35 0" rpy="0 0 0"/>
+    <origin xyz="-0.45 0.0 0" rpy="0 0 0"/>
     <child link="back_left_wheel"/>
-    <parent link="chassis"/>
-    <axis xyz="0 1 0" rpy="0 0 0"/>
-    <limit effort="10000" velocity="1000"/>
-    <dynamics damping="1.0" friction="1.0"/>
-  </joint>
-  <joint type="continuous" name="back_right_wheel_hinge">
-    <origin xyz="-0.45 -0.35 0" rpy="0 0 0"/>
-    <child link="back_right_wheel"/>
     <parent link="chassis"/>
     <axis xyz="0 1 0" rpy="0 0 0"/>

Commit message: SLAM

File: src/my_robot/urdf/my_robot.xacro (robot description, xacro)
@@ -253,4 +253,11 @@
     <axis xyz="0 1 0" rpy="0 0 0"/>
   </joint>
+  <joint name="camera_optical_joint" type="fixed">
+    <origin xyz="0 0 0" rpy="-1.5707 0 -1.5707"/>
+    <parent link="camera"/>
+    <child link="camera_link_optical"/>
+  </joint>
+  <link name="camera_link_optical">
+  </link>
 <link name='hokuyo'>
     <inertial>
